File: KiCAD/PC8001extRS232.sch (KiCad schematic (older format))
At the start: 32 parts, among them J1 PC8001 Ext Con, J2 232C JP, J3 232C-1, J4 232C-2, U1 74LS04, U10 74HC4060, U2 74LS148, U3 74LS541, U4 74LS32, U5 74LS04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

Commit message: アドレスデコーダ変更、割り込み回路のNOT削除
Parts:
- removed C10, C7: 0.1u, symbol Device:C_Small
- removed U5: 74LS04, symbol 74xx:74LS04
- removed U6: 74LS30, symbol 74xx:74LS30
- removed U7: 74LS32, symbol 74xx:74LS32
- added C9: 0.1u, symbol Device:C_Small
- added J5: INTJP, symbol Connector_Generic:Conn_01x06
- added U5: 74LS00, symbol 74xx:74LS00
- added U6: 74LS138, symbol 74HC4060:74LS138
- renumbered C8 to C7, C9 to C8, U8 to U7, U9 to U8, U10 to U9
Connections:
- wire segments 356 -> 331
- no-connect marks 42 -> 50
Other:
- note added: "~INT0"
- note added: "~INT1"
- note added: "~INT4"
- note added: "~INT5"
- note added: "~INT6"
- note added: "~INT7"
- moved on the sheet: C3, C7, C8, J1, J3, J4, R1, R2, RN2, U1A, U1B, U1C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

Commit message: プリント基板 REV1 ガーバー出力
Parts:
- added H1, H2, H3, H4: MountingHole, MountingHole:MountingHole_3.2mm_M3, symbol Mechanical:MountingHole
- C1, C11, C12, C2, C3, C4, C5, C6, C7, C8, C9: footprint (none) -> Capacitor_THT:C_Disc_D3.0mm_W1.6mm_P2.50mm
- J1: footprint (none) -> Connector_PinHeader_2.54mm:PinHeader_2x25_P2.54mm_Horizontal
- J2: footprint (none) -> Connector_PinHeader_2.54mm:PinHeader_2x06_P2.54mm_Vertical
- J3, J4, J5: footprint (none) -> Connector_PinHeader_2.54mm:PinHeader_1x06_P2.54mm_Horizontal
- R1, R2, R3: footprint (none) -> Resistor_THT:R_Axial_DIN0207_L6.3mm_D2.5mm_P10.16mm_Horizontal
- U1, U4, U5: footprint (none) -> Package_DIP:DIP-14_W7.62mm_Socket_LongPads
- U2, U6, U9: footprint (none) -> Package_DIP:DIP-16_W7.62mm_Socket_LongPads
- U3: footprint (none) -> Package_DIP:DIP-20_W7.62mm_Socket_LongPads
- U7, U8: footprint (none) -> Package_DIP:DIP-28_W15.24mm_Socket_LongPads
- Y1: footprint (none) -> Crystal:Crystal_HC49-U_Vertical
